File: KiCad/USBC-Lane1.kicad_sch (KiCad schematic)
At the start: 34 parts, among them J2 USB-C-MLX

Commit message: WiP layout
Parts:
- removed TP10: TPTP38X20, pcie2usbc:TP38X20, symbol pcie2usbc-eagle-import:TPTP38X20
- J2: footprint pcie2usbc:MOLEX_105450-0101 -> Connector_USB:USB_C_Receptacle_CNCTech_C-ARA1-AK51X
- R1, R10, R2, R3, R4, R5, R6, R7, R8: footprint pcie2usbc:R0603 -> Resistor_SMD:R_0402_1005Metric_Pad0.72x0.64mm_HandSolder
- TP13: footprint pcie2usbc:TP38X20 -> TestPoint:TestPoint_Pad_D1.5mm
- TP15: renamed from TP32; footprint TestPoint:TestPoint_Pad_D2.0mm -> TestPoint:TestPoint_Pad_1.0x1.0mm
- TP16: renamed from TP34; footprint TestPoint:TestPoint_Pad_D2.0mm -> TestPoint:TestPoint_Pad_1.0x1.0mm
- TP17: renamed from TP36; footprint TestPoint:TestPoint_Pad_D2.0mm -> TestPoint:TestPoint_Pad_1.0x1.0mm
- TP18: renamed from TP38; footprint TestPoint:TestPoint_Pad_D2.0mm -> TestPoint:TestPoint_Pad_1.0x1.0mm

Commit message: Final rework
Layout completed finally
Parts:
- removed TP13: TPTP38X20, TestPoint:TestPoint_Pad_D1.5mm, symbol pcie2usbc-eagle-import:TPTP38X20
- added GND1: TestPoint, TestPoint:TestPoint_Keystone_5015_Micro-Minature, symbol Connector:TestPoint
- J2: footprint Connector_USB:USB_C_Receptacle_CNCTech_C-ARA1-AK51X -> Connector_USB:USB_C_Receptacle_Amphenol_12401610E4-2A
- renumbered TP15 to TP16, TP16 to TP17, TP17 to TP18, TP18 to TP19
Connections:
- net GND: now also GND1.1
- net at C9.1, J2.S1 (SHIELD), R1.2: no longer J2.S2 (SHIELD), J2.S3 (SHIELD), J2.S4 (SHIELD)
Other:
- moved on the sheet: C1, C16, C17, C2, C3, C4, C5, C6, C7, C8, C9, J2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
