File: KiCad/pcie2usbc.kicad_sch (KiCad schematic)
At the start: 13 parts, among them J3 Bus_PCI_Express_x4, J4 Conn_02x05_Top_Bottom

Commit message: WiP layout
Parts:
- removed TP16, TP17, TP18, TP19, TP20, TP21, TP22, TP23, TP24: TestPoint, TestPoint:TestPoint_Pad_D2.0mm, symbol Connector:TestPoint
- R1: renamed from R10; footprint pcie2usbc:R0603 -> Resistor_SMD:R_0402_1005Metric_Pad0.72x0.64mm_HandSolder
- R2: renamed from R12; footprint pcie2usbc:R0603 -> Resistor_SMD:R_0402_1005Metric_Pad0.72x0.64mm_HandSolder
- renumbered J3 to J1, J4 to J2

Commit message: Final rework
Layout completed finally
Parts:
- removed J2: Conn_02x05_Top_Bottom, Connector_PinHeader_2.54mm:PinHeader_2x05_P2.54mm_Vertical, symbol Connector_Generic:Conn_02x05_Top_Bottom
- added TP1, TP10, TP2, TP3, TP4, TP5, TP6, TP7, TP8, TP9: TestPoint_Small, TestPoint:TestPoint_Pad_D1.0mm, symbol Connector:TestPoint_Small
- renumbered R2 to JP1, R1 to JP2
Connections:
- net CLKREQ_N: now also TP9.1
- net PRSNT2: no longer J1.B17 (~{PRSNT2})
- net SMCLK: now also TP1.1
- net SMDAT: now also TP3.1
- net TCK: now also TP2.1
- net TDI: now also TP4.1
- net TDO: now also TP6.1
- net TMS: now also TP8.1
- net TRST_N: now also TP5.1
- net VBUS_H: now also TP10.1
- net WAKE_N: now also TP7.1
- no-connect marks 3 -> 4
